Commit message: Remove Gazebo from the Husky description and use real wheel joint states, plus add navigation rviz configuration and add robot sizes for navigation aim

File: husky_a100_description/urdf/husky_a100.urdf.xacro (robot description, xacro)
@@ -16,5 +16,4 @@
     dimensions_file  file YAML delle dimensioni
     urdf_extras      file xacro aggiuntivo (sensori)
-    use_gazebo       true per includere i plugin di Gazebo Fortress
 -->
 <robot name="husky_a100" xmlns:xacro="http://ros.org/wiki/xacro">
@@ -23,5 +22,4 @@
   <xacro:arg name="dimensions_file" default=""/>
   <xacro:arg name="urdf_extras" default=""/>
-  <xacro:arg name="use_gazebo" default="false"/>
   <xacro:property name="_dims_arg" value="$(arg dimensions_file)"/>
   <xacro:property name="_extras_arg" value="$(arg urdf_extras)"/>
@@ -61,5 +59,4 @@
   <xacro:property name="mesh_d" value="${dims['mesh']['wheel_native_diameter']}"/>
   <xacro:property name="mesh_w" value="${dims['mesh']['wheel_native_width']}"/>
-  <xacro:property name="gz" value="${dims['gazebo']}"/>
   <xacro:include filename="materials.urdf.xacro"/>
   <xacro:include filename="wheel.urdf.xacro"/>
@@ -80,7 +77,5 @@
   <xacro:macro name="wheel_at" params="prefix x y mimic:=''">
     <xacro:a100_wheel prefix="${prefix}" x="${x}" y="${y}" radius="${r}" width="${w}" mass="${m_wheel}"
-                      mesh_file="${wheel_mesh}" mesh_d="${mesh_d}" mesh_w="${mesh_w}"
-                      mu1="${gz['wheel_mu1']}" mu2="${gz['wheel_mu2']}"
-                      kp="${gz['wheel_kp']}" kd="${gz['wheel_kd']}" mimic="${mimic}"/>
+                      mesh_file="${wheel_mesh}" mesh_d="${mesh_d}" mesh_w="${mesh_w}" mimic="${mimic}"/>
   </xacro:macro>
   <xacro:wheel_at prefix="front_left" x="${s}" y="${T / 2.0}"/>
@@ -90,8 +85,4 @@
   <xacro:wheel_at prefix="middle_right" x="0" y="${-T / 2.0}" mimic="front_right_wheel_joint"/>
   <xacro:wheel_at prefix="rear_right" x="${-s}" y="${-T / 2.0}"/>
-  <xacro:if value="$(arg use_gazebo)">
-    <xacro:include filename="gazebo.urdf.xacro"/>
-    <xacro:a100_gazebo/>
-  </xacro:if>
   <xacro:include filename="${extras_file}"/>
 </robot>

File: husky_a100_description/urdf/wheel.urdf.xacro (robot description, xacro)
@@ -17,5 +17,5 @@
 -->
 <robot xmlns:xacro="http://ros.org/wiki/xacro">
-  <xacro:macro name="a100_wheel" params="prefix x y radius width mass mesh_file mesh_d mesh_w mu1 mu2 kp kd mimic:=''">
+  <xacro:macro name="a100_wheel" params="prefix x y radius width mass mesh_file mesh_d mesh_w mimic:=''">
     <link name="${prefix}_wheel_link">
       <inertial>
@@ -40,12 +40,4 @@
       </collision>
     </link>
-    <!-- Parametri di contatto ripresi dalla macro noetic (usati solo da Gazebo) -->
-    <gazebo reference="${prefix}_wheel_link">
-      <mu1>${mu1}</mu1>
-      <mu2>${mu2}</mu2>
-      <kp>${kp}</kp>
-      <kd>${kd}</kd>
-      <fdir1>1 0 0</fdir1>
-    </gazebo>
     <joint name="${prefix}_wheel_joint" type="continuous">
       <parent link="base_link"/>
